File: windmill pcb.sch (KiCad schematic (older format))
At the start: 5 parts, among them M1 Stepper_Motor_bipolar

Commit message: Add files via upload
Parts:
- D1, D2: footprint (none) -> Diodes_THT:Diode_Bridge_DIP-4_W7.62mm_P5.08mm
Changed lines of the file:
@@
 F 0 "D1" H 4794 1696 50  0000 L CNN
 F 1 "Bridge Rectifier " H 4794 1605 50  0000 L CNN
-F 2 "" H 4450 1650 50  0001 C CNN
+F 2 "Diodes_THT:Diode_Bridge_DIP-4_W7.62mm_P5.08mm" H 4450 1650 50  0001 C CNN
 F 3 "~" H 4450 1650 50  0001 C CNN
 	1    4450 1650
@@
 F 0 "D2" H 4844 4196 50  0000 L CNN
 F 1 "Bridge Rectifier" H 4844 4105 50  0000 L CNN
-F 2 "" H 4500 4150 50  0001 C CNN
+F 2 "Diodes_THT:Diode_Bridge_DIP-4_W7.62mm_P5.08mm" H 4500 4150 50  0001 C CNN
 F 3 "~" H 4500 4150 50  0001 C CNN
 	1    4500 4150
